Commit message: 色々弄ってNavigationを除きGazeboで動くようになりました

File: lightrover_description/urdf/lidar/lidar_gazebo.xacro (robot description, xacro)
@@ -27,5 +27,5 @@
           </noise>
 		</ray>
-		<plugin name="gazebo_ros_${prefix}_lidar_controller" filename="libgazebo_ros_laser.so">
+		<plugin name="gazebo_ros_${prefix}_lidar_controller" filename="libgazebo_ros_ray_sensor.so">
           <topicName>/scan</topicName>
           <frameName>laser_frame</frameName>

File: lightrover_description/urdf/lightrover_urdf.xacro (robot description, xacro)
@@ -10,33 +10,54 @@
   <link name="base_footprint"/>
   <xacro:base parent="base_footprint">
-	  <origin xyz="0 0 0.024"/>
+    <origin xyz="0 0 0.024"/>
   </xacro:base>
   <!-- Caster -->
   <xacro:caster parent="base_link">
-	  <origin xyz="-0.078 0 -0.014"/>
+    <origin xyz="-0.078 0 -0.014"/>
   </xacro:caster>
   <!-- Wheel -->
   <!-- Right Wheel -->
   <xacro:wheel prefix="right" parent="base_link">
-	  <origin xyz="0 -0.072 0.006"/>
-	  <axis xyz="0 1 0"/>
+    <origin xyz="0 -0.072 0.006"/>
+    <axis xyz="0 1 0"/>
   </xacro:wheel>
   <!-- Left Wheel -->
   <xacro:wheel prefix="left" parent="base_link">
-	  <origin xyz="0 0.072 0.006" rpy="0 0 ${M_PI}"/>
-	  <axis xyz="0 -1 0"/>
+    <origin xyz="0 0.072 0.006" rpy="0 0 ${M_PI}"/>
+    <axis xyz="0 -1 0"/>
   </xacro:wheel>
   <!-- Sensors -->
   <!-- Lidar -->
   <xacro:lidar prefix="center" parent="base_link">
-  	<origin xyz="-0.07 0 0.086" rpy="0 0 -1.5708"/>
+    <origin xyz="-0.07 0 0.086" rpy="0 0 -1.5708"/>
   </xacro:lidar>
   <!-- ===============  Transmission =============== -->
   <xacro:wheel_trans prefix="right"/>
   <xacro:wheel_trans prefix="left"/>
+  <!-- =============== ros2_control =============== -->
+  <!-- ROS2 control 定義：GazeboSystem を使って2輪を速度制御 -->
+  <ros2_control name="GazeboSystem" type="system">
+    <hardware>
+      <plugin>gazebo_ros2_control/GazeboSystem</plugin>
+    </hardware>
+    <!-- 右車輪 -->
+    <joint name="right_wheel_joint">
+      <command_interface name="velocity"/>
+      <state_interface   name="position"/>
+      <state_interface   name="velocity"/>
+    </joint>
+    <!-- 左車輪 -->
+    <joint name="left_wheel_joint">
+      <command_interface name="velocity"/>
+      <state_interface   name="position"/>
+      <state_interface   name="velocity"/>
+    </joint>
+  </ros2_control>
   <!-- =============== Gazebo =============== -->
   <gazebo>
-    <plugin name="gazebo_ros_control" filename="libgazebo_ros_control.so">
-      <robotNamespace>lightrover</robotNamespace>
+    <!-- ROS2 用の ros2_control プラグイン -->
+    <plugin name="gazebo_ros2_control" filename="libgazebo_ros2_control.so">
+      <!-- コントローラ設定ファイル（xacro の $(find ...) は使えます） -->
+      <parameters>$(find lightrover_description)/config/lightrover_controllers.yaml</parameters>
     </plugin>
   </gazebo>
@@ -48,5 +69,5 @@
   <!-- LiDAR -->
   <xacro:lidar_gazebo prefix="center"
-					   min_rad="-${M_PI}" max_rad="${M_PI}"
-					   min_range="0.10" max_range="8.0"/>
+           min_rad="-${M_PI}" max_rad="${M_PI}"
+           min_range="0.10" max_range="8.0"/>
 </robot>
